Commit message: fixed lidar

File: leo_description/urdf/leo_sim.urdf.xacro (robot description, xacro)
@@ -5,4 +5,9 @@
   <xacro:arg name="robot_ns" default=""/>
   <xacro:arg name="mecanum_wheels" default="false"/>
+  <!-- Calculate the link prefix based on robot_ns -->
+  <xacro:property name="link_prefix" value=""/>
+  <xacro:if value="${'$(arg robot_ns)' != '' and '$(arg robot_ns)' != '/'}">
+    <xacro:property name="link_prefix" value="$(arg robot_ns)/"/>
+  </xacro:if>
   <xacro:include filename="$(find leo_description)/urdf/macros.xacro"/>
   <xacro:include filename="$(find leo_description)/urdf/lidar.urdf.xacro"/>
